File: RPi_shield/_saved_RPi_shield.sch (KiCad schematic (older format))
At the start: 16 parts, among them P1 CONN_BUTTON, P2 CONN_MOT_SEN_L, P3 CONN_MOT_SEN_R, P4 CONN_02X20, Q1 BC337, Q2 BC337

Commit message: Routage in progress
Parts:
- D1, D2: footprint (none) -> Diodes_THT:Diode_DO-41_SOD81_Horizontal_RM10
- P1: footprint (none) -> Pin_Headers:Pin_Header_Straight_1x02
- P2, P3: footprint (none) -> Pin_Headers:Pin_Header_Straight_1x06
- P4: footprint (none) -> Socket_Strips:Socket_Strip_Straight_2x20
- P5: renamed from P?; footprint (none) -> Pin_Headers:Pin_Header_Straight_1x03
- Q1, Q2: footprint TO-92 -> TO_SOT_Packages_THT:TO-92_Inline_Wide
- R1, R2, R3, R4, R5, R6, R7: footprint (none) -> Resistors_THT:Resistor_Horizontal_RM7mm
Changed lines of the file:
@@
 F 0 "Q1" H 3050 2875 50  0000 L CNN
 F 1 "BC337" H 3050 2800 50  0000 L CNN
-F 2 "TO-92" H 3050 2725 50  0000 L CIN
+F 2 "TO_SOT_Packages_THT:TO-92_Inline_Wide" H 3050 2725 50  0000 L CIN
 F 3 "" H 2850 2800 50  0000 L CNN
 	1    2850 2800
@@
 F 0 "R1" V 2580 2800 50  0000 C CNN
 F 1 "330" V 2500 2800 50  0000 C CNN
-F 2 "" V 2430 2800 50  0000 C CNN
+F 2 "Resistors_THT:Resistor_Horizontal_RM7mm" V 2430 2800 50  0001 C CNN
 F 3 "" H 2500 2800 50  0000 C CNN
 	1    2500 2800
@@
 F 0 "D1" H 3550 2900 50  0000 C CNN
 F 1 "1N4001" H 3550 2700 50  0000 C CNN
-F 2 "" H 3550 2800 50  0000 C CNN
+F 2 "Diodes_THT:Diode_DO-41_SOD81_Horizontal_RM10" H 3550 2800 50  0001 C CNN
 F 3 "" H 3550 2800 50  0000 C CNN
 	1    3550 2800
@@
 F 0 "R5" V 3580 4100 50  0000 C CNN
 F 1 "330" V 3500 4100 50  0000 C CNN
-F 2 "" V 3430 4100 50  0000 C CNN
+F 2 "Resistors_THT:Resistor_Horizontal_RM7mm" V 3430 4100 50  0001 C CNN
 F 3 "" H 3500 4100 50  0000 C CNN
 	1    3500 4100
@@
 F 0 "R3" V 3430 3300 50  0000 C CNN
 F 1 "1K" V 3350 3300 50  0000 C CNN
-F 2 "" V 3280 3300 50  0000 C CNN
+F 2 "Resistors_THT:Resistor_Horizontal_RM7mm" V 3280 3300 50  0001 C CNN
 F 3 "" H 3350 3300 50  0000 C CNN
 	1    3350 3300
@@
 F 0 "R7" V 3380 1450 50  0000 C CNN
 F 1 "1K" V 3300 1450 50  0000 C CNN
-F 2 "" V 3230 1450 50  0000 C CNN
+F 2 "Resistors_THT:Resistor_Horizontal_RM7mm" V 3230 1450 50  0001 C CNN
 F 3 "" H 3300 1450 50  0000 C CNN
 	1    3300 1450
@@
 F 0 "P2" H 1450 4000 50  0000 C CNN
 F 1 "CONN_MOT_SEN_L" V 1550 3650 50  0000 C CNN
-F 2 "" H 1450 3650 50  0000 C CNN
+F 2 "Pin_Headers:Pin_Header_Straight_1x06" H 1450 3650 50  0001 C CNN
 F 3 "" H 1450 3650 50  0000 C CNN
 	1    1450 3650
@@
 F 0 "P1" H 1450 1550 50  0000 C CNN
 F 1 "CONN_BUTTON" V 1550 1400 50  0000 C CNN
-F 2 "" H 1450 1400 50  0000 C CNN
+F 2 "Pin_Headers:Pin_Header_Straight_1x02" H 1450 1400 50  0001 C CNN
 F 3 "" H 1450 1400 50  0000 C CNN
 	1    1450 1400
@@
 F 0 "P4" H 10000 4650 50  0000 C CNN
 F 1 "CONN_02X20" V 10000 3600 50  0000 C CNN
-F 2 "" H 10000 2650 50  0000 C CNN
+F 2 "Socket_Strips:Socket_Strip_Straight_2x20" H 10000 2650 50  0001 C CNN
 F 3 "" H 10000 2650 50  0000 C CNN
 	1    10000 3600
@@
 F 0 "P3" H 1400 6550 50  0000 C CNN
 F 1 "CONN_MOT_SEN_R" V 1500 6200 50  0000 C CNN
-F 2 "" H 1400 6200 50  0000 C CNN
+F 2 "Pin_Headers:Pin_Header_Straight_1x06" H 1400 6200 50  0001 C CNN
 F 3 "" H 1400 6200 50  0000 C CNN
 	1    1400 6200
@@
 F 0 "Q2" H 3050 5725 50  0000 L CNN
 F 1 "BC337" H 3050 5650 50  0000 L CNN
-F 2 "TO-92" H 3050 5575 50  0000 L CIN
+F 2 "TO_SOT_Packages_THT:TO-92_Inline_Wide" H 3050 5575 50  0000 L CIN
 F 3 "" H 2850 5650 50  0000 L CNN
 	1    2850 5650
@@
 F 0 "R2" V 2580 5650 50  0000 C CNN
 F 1 "330" V 2500 5650 50  0000 C CNN
-F 2 "" V 2430 5650 50  0000 C CNN
+F 2 "Resistors_THT:Resistor_Horizontal_RM7mm" V 2430 5650 50  0001 C CNN
 F 3 "" H 2500 5650 50  0000 C CNN
 	1    2500 5650
@@
 F 0 "D2" H 3550 5750 50  0000 C CNN
 F 1 "1N4001" H 3550 5550 50  0000 C CNN
-F 2 "" H 3550 5650 50  0000 C CNN
+F 2 "Diodes_THT:Diode_DO-41_SOD81_Horizontal_RM10" H 3550 5650 50  0001 C CNN
 F 3 "" H 3550 5650 50  0000 C CNN
 	1    3550 5650
@@
 F 0 "R6" V 3580 6950 50  0000 C CNN
 F 1 "330" V 3500 6950 50  0000 C CNN
-F 2 "" V 3430 6950 50  0000 C CNN
+F 2 "Resistors_THT:Resistor_Horizontal_RM7mm" V 3430 6950 50  0001 C CNN
 F 3 "" H 3500 6950 50  0000 C CNN
 	1    3500 6950
@@
 F 0 "R4" V 3430 6150 50  0000 C CNN
 F 1 "1K" V 3350 6150 50  0000 C CNN
-F 2 "" V 3280 6150 50  0000 C CNN
+F 2 "Resistors_THT:Resistor_Horizontal_RM7mm" V 3280 6150 50  0001 C CNN
 F 3 "" H 3350 6150 50  0000 C CNN
 	1    3350 6150
@@
 NoConn ~ 9750 3450
 $Comp
-L +3.3V #PWR?
+L +3.3V #PWR015
 U 1 1 5862C9F2
 P 9750 2650
-F 0 "#PWR?" H 9750 2500 50  0001 C CNN
+F 0 "#PWR015" H 9750 2500 50  0001 C CNN
 F 1 "+3.3V" H 9750 2790 50  0000 C CNN
 F 2 "" H 9750 2650 50  0000 C CNN
@@
 RPI_BUTTON
 $Comp
-L +5V #PWR?
+L +5V #PWR016
 U 1 1 5862CDEF
 P 10250 2650
-F 0 "#PWR?" H 10250 2500 50  0001 C CNN
+F 0 "#PWR016" H 10250 2500 50  0001 C CNN
 F 1 "+5V" H 10250 2790 50  0000 C CNN
 F 2 "" H 10250 2650 50  0000 C CNN
@@
 $EndComp
 $Comp
-L GND #PWR?
+L GND #PWR017
 U 1 1 5862CE43
 P 10250 2850
-F 0 "#PWR?" H 10250 2600 50  0001 C CNN
+F 0 "#PWR017" H 10250 2600 50  0001 C CNN
 F 1 "GND" H 10250 2700 50  0000 C CNN
 F 2 "" H 10250 2850 50  0000 C CNN
@@
 OUT_SENSOR_L
 $Comp
-L CONN_01X03 P?
+L CONN_01X03 P5
 U 1 1 5862D92F
 P 6650 1900
-F 0 "P?" H 6650 2100 50  0000 C CNN
+F 0 "P5" H 6650 2100 50  0000 C CNN
 F 1 "CONN_01X03" V 6750 1900 50  0000 C CNN
-F 2 "" H 6650 1900 50  0000 C CNN
+F 2 "Pin_Headers:Pin_Header_Straight_1x03" H 6650 1900 50  0001 C CNN
 F 3 "" H 6650 1900 50  0000 C CNN
 	1    6650 1900
@@
 $EndComp
 $Comp
-L +3.3V #PWR?
+L +3.3V #PWR018
 U 1 1 5862D9D2
 P 6850 1800
-F 0 "#PWR?" H 6850 1650 50  0001 C CNN
+F 0 "#PWR018" H 6850 1650 50  0001 C CNN
 F 1 "+3.3V" H 6850 1940 50  0000 C CNN
 F 2 "" H 6850 1800 50  0000 C CNN
@@
 $EndComp
 $Comp
-L GND #PWR?
+L GND #PWR019
 U 1 1 5862DA06
 P 6850 2000
-F 0 "#PWR?" H 6850 1750 50  0001 C CNN
+F 0 "#PWR019" H 6850 1750 50  0001 C CNN
 F 1 "GND" H 6850 1850 50  0000 C CNN
 F 2 "" H 6850 2000 50  0000 C CNN
